File: conveyor-design-files/pcb-files/conveyor-pcb.brd (EAGLE design)
At the start: 100 x 53 mm, 28 parts

Commit message: updates to pcb files
Parts:
- removed C1: 100uF, SparkFun-Capacitors:CPOL-RADIAL-2.5MM-6.5MM
- added U$20: CAP_100UF, Capacitor:CAP_100UF
Connections:
- net +5V: now also U$20.+5V; no longer C1.1
- net GND: now also U$20.GND; no longer C1.2
Changed lines of the file:
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@@
 <?xml version="1.0" encoding="utf-8"?>
 <!DOCTYPE eagle SYSTEM "eagle.dtd">
-<!-- Copyright 2018 Amazon.com, Inc. or its affiliates. All Rights Reserved. -->
-<!-- SPDX-License-Identifier: Apache-2.0 -->
 <eagle version="8.2.2">
 <drawing>
@@
 <element name="5V_POWER" library="ScrewTerminals" package="2.54MM_2P" value="2.54MM_2P" x="83.82" y="6.35" smashed="yes" rot="R180"/>
 <element name="ACCELEROMETER" library="Adafruit" package="ADAFRUIT_ADXL335" value="ADAFRUIT_ADXL335" x="24.13" y="25.4" smashed="yes" rot="R270"/>
-<element name="C1" library="SparkFun-Capacitors" package="CPOL-RADIAL-2.5MM-6.5MM" value="100uF" x="69.85" y="5.08" smashed="yes" rot="R90">
-<attribute name="PROD_ID" value="CAP-08439" x="69.85" y="5.08" size="1.778" layer="27" rot="R90" display="off"/>
-</element>
 <element name="RPM_SENSOR" library="ScrewTerminals" package="2.54MM_3P" value="2.54MM_3P" x="12.7" y="34.29" smashed="yes" rot="R270"/>
 <element name="SENSOR" library="ScrewTerminals" package="2.54MM_3P" value="2.54MM_3P" x="83.82" y="26.67" smashed="yes" rot="R180"/>
@@
 <element name="U$18" library="Headers" package="1PIN_HEADER" value="1PIN_HEADER" x="76.2" y="26.67"/>
 <element name="U$19" library="Headers" package="1PIN_HEADER" value="1PIN_HEADER" x="76.2" y="29.21"/>
+<element name="U$20" library="Capacitor" package="CAP_100UF" value="CAP_100UF" x="69.85" y="5.08" rot="R270"/>
 </elements>
 <signals>
@@
 <contactref element="SENSOR" pad="P$2"/>
 <contactref element="5V_POWER" pad="P$1"/>
-<contactref element="C1" pad="2"/>
 <contactref element="STEPPER_CONTROL" pad="GND@1"/>
 <contactref element="STEPPER_CONTROL" pad="GND@2"/>
@@
 <contactref element="U$18" pad="P$1"/>
 <contactref element="U$12" pad="P$1"/>
+<contactref element="U$20" pad="GND"/>
 </signal>
 <signal name="EN">
@@
 <signal name="+5V">
 <contactref element="5V_POWER" pad="P$2"/>
-<contactref element="C1" pad="1"/>
 <contactref element="STEPPER_CONTROL" pad="VMOT"/>
 <contactref element="U$2" pad="P$1"/>
 <contactref element="ESP1" pad="VIN5V"/>
-<wire x1="83.82" y1="8.89" x2="72.41" y2="8.89" width="1.016" layer="1"/>
 <wire x1="73.66" y1="29.0767125" x2="73.66" y2="29.21" width="1.016" layer="1"/>
 <contactref element="U$19" pad="P$1"/>
@@
 <wire x1="73.66" y1="29.21" x2="71.12" y2="29.21" width="1.016" layer="1"/>
 <wire x1="71.12" y1="29.21" x2="69.85" y2="27.94" width="1.016" layer="1"/>
-<wire x1="72.41" y1="8.89" x2="69.85" y2="6.33" width="1.016" layer="1"/>
-<wire x1="66.825834375" y1="6.33" x2="69.85" y2="6.33" width="1.016" layer="1"/>
 <wire x1="66.825834375" y1="6.33" x2="58.908" y2="6.33" width="1.016" layer="1"/>
 <wire x1="58.908" y1="6.33" x2="54.1274" y2="1.5494" width="1.016" layer="1"/>
@@
 <wire x1="69.85" y1="9.354165625" x2="66.825834375" y2="6.33" width="1.016" layer="1"/>
 <wire x1="69.85" y1="27.94" x2="69.85" y2="9.354165625" width="1.016" layer="1"/>
+<contactref element="U$20" pad="+5V"/>
+<wire x1="72.39" y1="8.89" x2="69.85" y2="6.35" width="1.016" layer="1"/>
+<wire x1="83.82" y1="8.89" x2="72.39" y2="8.89" width="1.016" layer="1"/>
+<wire x1="69.85" y1="6.35" x2="66.845834375" y2="6.35" width="1.016" layer="1"/>
+<wire x1="66.845834375" y1="6.35" x2="66.825834375" y2="6.33" width="1.016" layer="1"/>
 </signal>
 <signal name="P$8">
