File: conveyor-design-files/pcb-files/conveyor-pcb.sch (EAGLE design)
At the start: 28 parts

Commit message: updates to pcb files
Parts:
- removed C1: 100uF, SparkFun-Capacitors:100UF-POLAR-RADIAL-2.5MM-25V-20%
- added U$20: CAP_100UF, Capacitor:CAP_100UF
Connections:
- net +5V: now also U$20.+5V; no longer C1.+
- net GND: now also U$20.GND; no longer C1.-
Changed lines of the file:
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@@
 <?xml version="1.0" encoding="utf-8"?>
 <!DOCTYPE eagle SYSTEM "eagle.dtd">
-<!-- Copyright 2018 Amazon.com, Inc. or its affiliates. All Rights Reserved. -->
-<!-- SPDX-License-Identifier: Apache-2.0 -->
 <eagle version="8.2.2">
 <drawing>
@@
 </classes>
 <parts>
-<part name="C1" library="SparkFun-Capacitors" deviceset="100UF-POLAR" device="-RADIAL-2.5MM-25V-20%" value="100uF"/>
 <part name="ACCELEROMETER" library="Adafruit" deviceset="ADAFRUIT_ADXL335" device=""/>
 <part name="U$1" library="19pinheader" deviceset="19PINHEADER" device=""/>
@@
 <part name="U$18" library="Headers" deviceset="1PIN_HEADER" device=""/>
 <part name="U$19" library="Headers" deviceset="1PIN_HEADER" device=""/>
+<part name="U$20" library="Capacitor" deviceset="CAP_100UF" device=""/>
 </parts>
 <sheets>
@@
 </plain>
 <instances>
-<instance part="C1" gate="G$1" x="124.46" y="5.08"/>
 <instance part="ACCELEROMETER" gate="G$1" x="99.06" y="-58.42"/>
 <instance part="U$1" gate="G$1" x="50.8" y="0"/>
@@
 <instance part="U$18" gate="G$1" x="133.985" y="0"/>
 <instance part="U$19" gate="G$1" x="133.985" y="7.62"/>
+<instance part="U$20" gate="G$1" x="127" y="5.08"/>
 </instances>
 <busses>
@@
 </segment>
 <segment>
-<pinref part="C1" gate="G$1" pin="-"/>
-<wire x1="124.46" y1="0" x2="133.985" y2="0" width="0.1524" layer="91"/>
+<wire x1="116.84" y1="0" x2="127" y2="0" width="0.1524" layer="91"/>
 <label x="127.635" y="-1.905" size="1.778" layer="95"/>
 <pinref part="STEPPER_CONTROL" gate="G$1" pin="GND@1"/>
-<wire x1="116.84" y1="0" x2="124.46" y2="0" width="0.1524" layer="91"/>
-<junction x="124.46" y="0"/>
 <pinref part="U$18" gate="G$1" pin="P$1"/>
+<pinref part="U$20" gate="G$1" pin="GND"/>
+<wire x1="127" y1="0" x2="133.985" y2="0" width="0.1524" layer="91"/>
+<junction x="127" y="0"/>
 </segment>
 <segment>
@@
 </segment>
 <segment>
-<pinref part="C1" gate="G$1" pin="+"/>
-<wire x1="124.46" y1="7.62" x2="133.985" y2="7.62" width="0.1524" layer="91"/>
+<wire x1="116.84" y1="7.62" x2="127" y2="7.62" width="0.1524" layer="91"/>
 <label x="128.905" y="7.62" size="1.778" layer="95"/>
 <pinref part="STEPPER_CONTROL" gate="G$1" pin="VMOT"/>
+<wire x1="127" y1="7.62" x2="133.985" y2="7.62" width="0.1524" layer="91"/>
 <wire x1="116.84" y1="5.08" x2="116.84" y2="7.62" width="0.1524" layer="91"/>
-<wire x1="116.84" y1="7.62" x2="124.46" y2="7.62" width="0.1524" layer="91"/>
-<junction x="124.46" y="7.62"/>
 <pinref part="U$19" gate="G$1" pin="P$1"/>
-</segment>
-<segment>
+<pinref part="U$20" gate="G$1" pin="+5V"/>
+<junction x="127" y="7.62"/>
+</segment>
+<segment>
